Commit message: oculus droid version 0: changed r to R as RG, LG is needed

File: anubis/urdf/anubis_v3.urdf (robot description, URDF)
Before this commit: robot anubis, 24 links, 23 joints
Joints:
- joint arm1_base_link_joint: limit lower=-2.41 upper=2.41 effort=39 velocity=1.3963 -> lower=-1.74533 upper=1.74533 effort=39 velocity=1.3963
- joint arm2_base_link_joint: limit lower=-2.41 upper=2.41 effort=39 velocity=1.3963 -> lower=-1.74533 upper=1.74533 effort=39 velocity=1.3963
- joint dummy_base_revolute_z_joint: limit lower=-360.0 upper=360.0 effort=100 velocity=100 -> lower=-6.283 upper=6.283 effort=100 velocity=100
- joint link11_joint: limit lower=-2.41 upper=2.41 effort=39 velocity=1.3963 -> lower=-0.523599 upper=0.523599 effort=39 velocity=1.3963
- joint link12_joint: limit lower=-2.41 upper=2.41 effort=39 velocity=1.3963 -> lower=-0.523599 upper=1.91986 effort=39 velocity=1.3963
- joint link13_joint: limit lower=-2.41 upper=2.41 effort=39 velocity=1.3963 -> lower=0.174533 upper=2.79253 effort=39 velocity=1.3963
- joint link14_joint: limit lower=-2.41 upper=2.41 effort=39 velocity=1.3963 -> lower=-1.5708 upper=1.74533 effort=39 velocity=1.3963
- joint link15_joint: limit lower=-2.41 upper=2.41 effort=39 velocity=1.3963 -> lower=-1.5708 upper=1.57085 effort=39 velocity=1.3963
- joint link21_joint: limit lower=-2.41 upper=2.41 effort=39 velocity=1.3963 -> lower=-0.523599 upper=0.523599 effort=39 velocity=1.3963
- joint link22_joint: limit lower=-2.41 upper=2.41 effort=39 velocity=1.3963 -> lower=-0.523599 upper=1.91986 effort=39 velocity=1.3963
- joint link23_joint: limit lower=-2.41 upper=2.41 effort=39 velocity=1.3963 -> lower=0.174533 upper=2.79253 effort=39 velocity=1.3963
- joint link24_joint: limit lower=-2.41 upper=2.41 effort=39 velocity=1.3963 -> lower=-1.5708 upper=1.74533 effort=39 velocity=1.3963
- joint link25_joint: limit lower=-2.41 upper=2.41 effort=39 velocity=1.3963 -> lower=-1.5708 upper=1.57085 effort=39 velocity=1.3963
