Commit message: omniwheel anubis

File: anubis/anubis_omni.urdf (robot description, URDF)
Before this commit: robot anubis, 24 links, 23 joints
Links:
- added link OmniFL_roller_0; collision sphere radius=0.03
- added link OmniFL_roller_1; collision sphere radius=0.03
- added link OmniFL_roller_2; collision sphere radius=0.03
- added link OmniFL_roller_3; collision sphere radius=0.03
- added link OmniFL_roller_4; collision sphere radius=0.03
- added link OmniFL_roller_5; collision sphere radius=0.03
- added link OmniFL_roller_6; collision sphere radius=0.03
- added link OmniFL_roller_7; collision sphere radius=0.03
- added link OmniFL_roller_8; collision sphere radius=0.03
- added link OmniFL_roller_9; collision sphere radius=0.03
- added link OmniFR_roller_0; collision sphere radius=0.03
- added link OmniFR_roller_1; collision sphere radius=0.03
- added link OmniFR_roller_2; collision sphere radius=0.03
- added link OmniFR_roller_3; collision sphere radius=0.03
- added link OmniFR_roller_4; collision sphere radius=0.03
- added link OmniFR_roller_5; collision sphere radius=0.03
- added link OmniFR_roller_6; collision sphere radius=0.03
- added link OmniFR_roller_7; collision sphere radius=0.03
- added link OmniFR_roller_8; collision sphere radius=0.03
- added link OmniFR_roller_9; collision sphere radius=0.03
- added link OmniR_roller_0; collision sphere radius=0.03
- added link OmniR_roller_1; collision sphere radius=0.03
- added link OmniR_roller_2; collision sphere radius=0.03
- added link OmniR_roller_3; collision sphere radius=0.03
- added link OmniR_roller_4; collision sphere radius=0.03
- added link OmniR_roller_5; collision sphere radius=0.03
- added link OmniR_roller_6; collision sphere radius=0.03
- added link OmniR_roller_7; collision sphere radius=0.03
- added link OmniR_roller_8; collision sphere radius=0.03
- added link OmniR_roller_9; collision sphere radius=0.03
- link OmniFL_wheel: geometry collision cylinder length=0.05 radius=0.029; collision cylinder length=0.05 radius=0.08
- link OmniFR_wheel: geometry collision cylinder length=0.05 radius=0.029; collision cylinder length=0.05 radius=0.08
- link OmniR_wheel: geometry collision cylinder length=0.05 radius=0.029; collision cylinder length=0.05 radius=0.08
Joints:
- added joint OmniFL_roller_0_joint: type continuous, parent OmniFL_wheel, child OmniFL_roller_0, origin xyz=0 0.073 0 rpy=0 0 0, axis 0 0 1
- added joint OmniFL_roller_1_joint: type continuous, parent OmniFL_wheel, child OmniFL_roller_1, origin xyz=0 0.0589 0.0430 rpy=0 0 0, axis 0 -0.588 0.809
- added joint OmniFL_roller_2_joint: type continuous, parent OmniFL_wheel, child OmniFL_roller_2, origin xyz=0 0.0225 0.07030  rpy=0 0 0, axis 0 -0.939 -0.343
- added joint OmniFL_roller_3_joint: type continuous, parent OmniFL_wheel, child OmniFL_roller_3, origin xyz=0 -0.0225 0.0703 rpy=0 0 0, axis 0 -0.939 -0.343
- added joint OmniFL_roller_4_joint: type continuous, parent OmniFL_wheel, child OmniFL_roller_4, origin xyz=0 -0.0589 0.0430 rpy=0 0 0, axis 0 -0.588 0.809
- added joint OmniFL_roller_5_joint: type continuous, parent OmniFL_wheel, child OmniFL_roller_5, origin xyz=0 -0.073 0 rpy=0 0 0, axis 0 0 1
- added joint OmniFL_roller_6_joint: type continuous, parent OmniFL_wheel, child OmniFL_roller_6, origin xyz=0 -0.0589 -0.0430 rpy=0 0 0, axis 0 0.588 -0.809
- added joint OmniFL_roller_7_joint: type continuous, parent OmniFL_wheel, child OmniFL_roller_7, origin xyz=0 -0.0225 -0.0703 rpy=0 0 0, axis 0 0.939 0.343
- added joint OmniFL_roller_8_joint: type continuous, parent OmniFL_wheel, child OmniFL_roller_8, origin xyz=0 0.0225 -0.0703 rpy=0 0 0, axis 0 0.939 0.343
- added joint OmniFL_roller_9_joint: type continuous, parent OmniFL_wheel, child OmniFL_roller_9, origin xyz=0 0.0589 -0.0430 rpy=0 0 0, axis 0 0.588 -0.809
- added joint OmniFR_roller_0_joint: type continuous, parent OmniFR_wheel, child OmniFR_roller_0, origin xyz=0 0.073 0 rpy=0 0 0, axis 0 0 1
- added joint OmniFR_roller_1_joint: type continuous, parent OmniFR_wheel, child OmniFR_roller_1, origin xyz=0 0.0589 0.0430 rpy=0 0 0, axis 0 -0.588 0.809
- added joint OmniFR_roller_2_joint: type continuous, parent OmniFR_wheel, child OmniFR_roller_2, origin xyz=0 0.0225 0.07030  rpy=0 0 0, axis 0 -0.939 -0.343
- added joint OmniFR_roller_3_joint: type continuous, parent OmniFR_wheel, child OmniFR_roller_3, origin xyz=0 -0.0225 0.0703 rpy=0 0 0, axis 0 -0.939 -0.343
- added joint OmniFR_roller_4_joint: type continuous, parent OmniFR_wheel, child OmniFR_roller_4, origin xyz=0 -0.0589 0.0430 rpy=0 0 0, axis 0 -0.588 0.809
- added joint OmniFR_roller_5_joint: type continuous, parent OmniFR_wheel, child OmniFR_roller_5, origin xyz=0 -0.073 0 rpy=0 0 0, axis 0 0 1
- added joint OmniFR_roller_6_joint: type continuous, parent OmniFR_wheel, child OmniFR_roller_6, origin xyz=0 -0.0589 -0.0430 rpy=0 0 0, axis 0 0.588 -0.809
- added joint OmniFR_roller_7_joint: type continuous, parent OmniFR_wheel, child OmniFR_roller_7, origin xyz=0 -0.0225 -0.0703 rpy=0 0 0, axis 0 0.939 0.343
- added joint OmniFR_roller_8_joint: type continuous, parent OmniFR_wheel, child OmniFR_roller_8, origin xyz=0 0.0225 -0.0703 rpy=0 0 0, axis 0 0.939 0.343
- added joint OmniFR_roller_9_joint: type continuous, parent OmniFR_wheel, child OmniFR_roller_9, origin xyz=0 0.0589 -0.0430 rpy=0 0 0, axis 0 0.588 -0.809
- added joint OmniR_roller_0_joint: type continuous, parent OmniR_wheel, child OmniR_roller_0, origin xyz=0 0.073 0 rpy=0 0 0, axis 0 0 1
- added joint OmniR_roller_1_joint: type continuous, parent OmniR_wheel, child OmniR_roller_1, origin xyz=0 0.0589 0.0430 rpy=0 0 0, axis 0 -0.588 0.809
- added joint OmniR_roller_2_joint: type continuous, parent OmniR_wheel, child OmniR_roller_2, origin xyz=0 0.0225 0.07030  rpy=0 0 0, axis 0 -0.939 -0.343
- added joint OmniR_roller_3_joint: type continuous, parent OmniR_wheel, child OmniR_roller_3, origin xyz=0 -0.0225 0.0703 rpy=0 0 0, axis 0 -0.939 -0.343
- added joint OmniR_roller_4_joint: type continuous, parent OmniR_wheel, child OmniR_roller_4, origin xyz=0 -0.0589 0.0430 rpy=0 0 0, axis 0 -0.588 0.809
- added joint OmniR_roller_5_joint: type continuous, parent OmniR_wheel, child OmniR_roller_5, origin xyz=0 -0.073 0 rpy=0 0 0, axis 0 0 1
- added joint OmniR_roller_6_joint: type continuous, parent OmniR_wheel, child OmniR_roller_6, origin xyz=0 -0.0589 -0.0430 rpy=0 0 0, axis 0 0.588 -0.809
- added joint OmniR_roller_7_joint: type continuous, parent OmniR_wheel, child OmniR_roller_7, origin xyz=0 -0.0225 -0.0703 rpy=0 0 0, axis 0 0.939 0.343
- added joint OmniR_roller_8_joint: type continuous, parent OmniR_wheel, child OmniR_roller_8, origin xyz=0 0.0225 -0.0703 rpy=0 0 0, axis 0 0.939 0.343
- added joint OmniR_roller_9_joint: type continuous, parent OmniR_wheel, child OmniR_roller_9, origin xyz=0 0.0589 -0.0430 rpy=0 0 0, axis 0 0.588 -0.809

Commit message: 1,2 fixed but by looking into the camera, movement is still be stable.
2. Make a stable wheel
3. Rotation of arm

File: anubis/anubis_omni.urdf (robot description, URDF)
Before this commit: robot anubis, 54 links, 53 joints
Joints:
- joint OmniFL_roller_0_joint: origin xyz=0 0.073 0 rpy=0 0 0 -> xyz=0 0.065 0.0 rpy=0 0 0
- joint OmniFL_roller_1_joint: origin xyz=0 0.0589 0.0430 rpy=0 0 0 -> xyz=0 0.0526 0.0380 rpy=0 0 0
- joint OmniFL_roller_2_joint: axis 0 -0.939 -0.343 -> 0 -0.940 0.342; origin xyz=0 0.0225 0.07030  rpy=0 0 0 -> xyz=0 0.0201 0.0617 rpy=0 0 0
- joint OmniFL_roller_3_joint: axis 0 -0.939 -0.343 -> 0 -0.940 -0.342; origin xyz=0 -0.0225 0.0703 rpy=0 0 0 -> xyz=0 -0.0201 0.0617 rpy=0 0 0
- joint OmniFL_roller_4_joint: axis 0 -0.588 0.809 -> 0 -0.588 -0.809; origin xyz=0 -0.0589 0.0430 rpy=0 0 0 -> xyz=0 -0.0526 0.0380 rpy=0 0 0
- joint OmniFL_roller_5_joint: axis 0 0 1 -> 0 0 -1; origin xyz=0 -0.073 0 rpy=0 0 0 -> xyz=0 -0.065 0.0 rpy=0 0 0
- joint OmniFL_roller_6_joint: origin xyz=0 -0.0589 -0.0430 rpy=0 0 0 -> xyz=0 -0.0526 -0.0380 rpy=0 0 0
- joint OmniFL_roller_7_joint: axis 0 0.939 0.343 -> 0 0.940 -0.342; origin xyz=0 -0.0225 -0.0703 rpy=0 0 0 -> xyz=0 -0.0201 -0.0617 rpy=0 0 0
- joint OmniFL_roller_8_joint: axis 0 0.939 0.343 -> 0 0.940 0.342; origin xyz=0 0.0225 -0.0703 rpy=0 0 0 -> xyz=0 0.0201 -0.0617 rpy=0 0 0
- joint OmniFL_roller_9_joint: axis 0 0.588 -0.809 -> 0 0.588 0.809; origin xyz=0 0.0589 -0.0430 rpy=0 0 0 -> xyz=0 0.0526 -0.0380 rpy=0 0 0
- joint OmniFR_roller_0_joint: origin xyz=0 0.073 0 rpy=0 0 0 -> xyz=0 0.065 0.0 rpy=0 0 0
- joint OmniFR_roller_1_joint: origin xyz=0 0.0589 0.0430 rpy=0 0 0 -> xyz=0 0.0526 0.0380 rpy=0 0 0
- joint OmniFR_roller_2_joint: axis 0 -0.939 -0.343 -> 0 -0.940 0.342; origin xyz=0 0.0225 0.07030  rpy=0 0 0 -> xyz=0 0.0201 0.0617 rpy=0 0 0
- joint OmniFR_roller_3_joint: axis 0 -0.939 -0.343 -> 0 -0.940 -0.342; origin xyz=0 -0.0225 0.0703 rpy=0 0 0 -> xyz=0 -0.0201 0.0617 rpy=0 0 0
- joint OmniFR_roller_4_joint: axis 0 -0.588 0.809 -> 0 -0.588 -0.809; origin xyz=0 -0.0589 0.0430 rpy=0 0 0 -> xyz=0 -0.0526 0.0380 rpy=0 0 0
- joint OmniFR_roller_5_joint: axis 0 0 1 -> 0 0 -1; origin xyz=0 -0.073 0 rpy=0 0 0 -> xyz=0 -0.065 0.0 rpy=0 0 0
- joint OmniFR_roller_6_joint: origin xyz=0 -0.0589 -0.0430 rpy=0 0 0 -> xyz=0 -0.0526 -0.0380 rpy=0 0 0
- joint OmniFR_roller_7_joint: axis 0 0.939 0.343 -> 0 0.940 -0.342; origin xyz=0 -0.0225 -0.0703 rpy=0 0 0 -> xyz=0 -0.0201 -0.0617 rpy=0 0 0
- joint OmniFR_roller_8_joint: axis 0 0.939 0.343 -> 0 0.940 0.342; origin xyz=0 0.0225 -0.0703 rpy=0 0 0 -> xyz=0 0.0201 -0.0617 rpy=0 0 0
- joint OmniFR_roller_9_joint: axis 0 0.588 -0.809 -> 0 0.588 0.809; origin xyz=0 0.0589 -0.0430 rpy=0 0 0 -> xyz=0 0.0526 -0.0380 rpy=0 0 0
- joint OmniR_roller_0_joint: origin xyz=0 0.073 0 rpy=0 0 0 -> xyz=0 0.065 0.0 rpy=0 0 0
- joint OmniR_roller_1_joint: origin xyz=0 0.0589 0.0430 rpy=0 0 0 -> xyz=0 0.0526 0.0380 rpy=0 0 0
- joint OmniR_roller_2_joint: axis 0 -0.939 -0.343 -> 0 -0.940 0.342; origin xyz=0 0.0225 0.07030  rpy=0 0 0 -> xyz=0 0.0201 0.0617 rpy=0 0 0
- joint OmniR_roller_3_joint: axis 0 -0.939 -0.343 -> 0 -0.940 -0.342; origin xyz=0 -0.0225 0.0703 rpy=0 0 0 -> xyz=0 -0.0201 0.0617 rpy=0 0 0
- joint OmniR_roller_4_joint: axis 0 -0.588 0.809 -> 0 -0.588 -0.809; origin xyz=0 -0.0589 0.0430 rpy=0 0 0 -> xyz=0 -0.0526 0.0380 rpy=0 0 0
- joint OmniR_roller_5_joint: axis 0 0 1 -> 0 0 -1; origin xyz=0 -0.073 0 rpy=0 0 0 -> xyz=0 -0.065 0.0 rpy=0 0 0
- joint OmniR_roller_6_joint: origin xyz=0 -0.0589 -0.0430 rpy=0 0 0 -> xyz=0 -0.0526 -0.0380 rpy=0 0 0
- joint OmniR_roller_7_joint: axis 0 0.939 0.343 -> 0 0.940 -0.342; origin xyz=0 -0.0225 -0.0703 rpy=0 0 0 -> xyz=0 -0.0201 -0.0617 rpy=0 0 0
- joint OmniR_roller_8_joint: axis 0 0.939 0.343 -> 0 0.940 0.342; origin xyz=0 0.0225 -0.0703 rpy=0 0 0 -> xyz=0 0.0201 -0.0617 rpy=0 0 0
- joint OmniR_roller_9_joint: axis 0 0.588 -0.809 -> 0 0.588 0.809; origin xyz=0 0.0589 -0.0430 rpy=0 0 0 -> xyz=0 0.0526 -0.0380 rpy=0 0 0
