Commit message: anubis with 20 spheres per wheel

File: anubis/anubis_omni.urdf (robot description, URDF)
Before this commit: robot anubis, 54 links, 53 joints
Links:
- added link OmniFL_roller_10, mass 0.05; collision sphere radius=0.03
- added link OmniFL_roller_11, mass 0.01; collision sphere radius=0.015
- added link OmniFL_roller_12, mass 0.05; collision sphere radius=0.03
- added link OmniFL_roller_13, mass 0.01; collision sphere radius=0.015
- added link OmniFL_roller_14, mass 0.05; collision sphere radius=0.03
- added link OmniFL_roller_15, mass 0.01; collision sphere radius=0.015
- added link OmniFL_roller_16, mass 0.05; collision sphere radius=0.03
- added link OmniFL_roller_17, mass 0.01; collision sphere radius=0.015
- added link OmniFL_roller_18, mass 0.05; collision sphere radius=0.03
- added link OmniFL_roller_19, mass 0.01; collision sphere radius=0.015
- added link OmniFR_roller_10, mass 0.05; collision sphere radius=0.03
- added link OmniFR_roller_11, mass 0.01; collision sphere radius=0.015
- added link OmniFR_roller_12, mass 0.05; collision sphere radius=0.03
- added link OmniFR_roller_13, mass 0.01; collision sphere radius=0.015
- added link OmniFR_roller_14, mass 0.05; collision sphere radius=0.03
- added link OmniFR_roller_15, mass 0.01; collision sphere radius=0.015
- added link OmniFR_roller_16, mass 0.05; collision sphere radius=0.03
- added link OmniFR_roller_17, mass 0.01; collision sphere radius=0.015
- added link OmniFR_roller_18, mass 0.05; collision sphere radius=0.03
- added link OmniFR_roller_19, mass 0.01; collision sphere radius=0.015
- added link OmniR_roller_10, mass 0.05; collision sphere radius=0.03
- added link OmniR_roller_11, mass 0.01; collision sphere radius=0.015
- added link OmniR_roller_12, mass 0.05; collision sphere radius=0.03
- added link OmniR_roller_13, mass 0.01; collision sphere radius=0.015
- added link OmniR_roller_14, mass 0.05; collision sphere radius=0.03
- added link OmniR_roller_15, mass 0.01; collision sphere radius=0.015
- added link OmniR_roller_16, mass 0.05; collision sphere radius=0.03
- added link OmniR_roller_17, mass 0.01; collision sphere radius=0.015
- added link OmniR_roller_18, mass 0.05; collision sphere radius=0.03
- added link OmniR_roller_19, mass 0.01; collision sphere radius=0.015
- link OmniFL_roller_0: mass None -> 0.05
- link OmniFL_roller_1: mass None -> 0.01; geometry collision sphere radius=0.015
- link OmniFL_roller_2: mass None -> 0.05
- link OmniFL_roller_3: mass None -> 0.01; geometry collision sphere radius=0.015
- link OmniFL_roller_4: mass None -> 0.05
- link OmniFL_roller_5: mass None -> 0.01; geometry collision sphere radius=0.015
- link OmniFL_roller_6: mass None -> 0.05
- link OmniFL_roller_7: mass None -> 0.01; geometry collision sphere radius=0.015
- link OmniFL_roller_8: mass None -> 0.05
- link OmniFL_roller_9: mass None -> 0.01; geometry collision sphere radius=0.015
- link OmniFR_roller_0: mass None -> 0.05
- link OmniFR_roller_1: mass None -> 0.01; geometry collision sphere radius=0.015
- link OmniFR_roller_2: mass None -> 0.05
- link OmniFR_roller_3: mass None -> 0.01; geometry collision sphere radius=0.015
- link OmniFR_roller_4: mass None -> 0.05
- link OmniFR_roller_5: mass None -> 0.01; geometry collision sphere radius=0.015
- link OmniFR_roller_6: mass None -> 0.05
- link OmniFR_roller_7: mass None -> 0.01; geometry collision sphere radius=0.015
- link OmniFR_roller_8: mass None -> 0.05
- link OmniFR_roller_9: mass None -> 0.01; geometry collision sphere radius=0.015
- link OmniR_roller_0: mass None -> 0.05
- link OmniR_roller_1: mass None -> 0.01; geometry collision sphere radius=0.015
- link OmniR_roller_2: mass None -> 0.05
- link OmniR_roller_3: mass None -> 0.01; geometry collision sphere radius=0.015
- link OmniR_roller_4: mass None -> 0.05
- link OmniR_roller_5: mass None -> 0.01; geometry collision sphere radius=0.015
- link OmniR_roller_6: mass None -> 0.05
- link OmniR_roller_7: mass None -> 0.01; geometry collision sphere radius=0.015
- link OmniR_roller_8: mass None -> 0.05
- link OmniR_roller_9: mass None -> 0.01; geometry collision sphere radius=0.015
- link base_link: mass 40 -> 30
Joints:
- added joint OmniFL_roller_10_joint: type continuous, parent OmniFL_wheel, child OmniFL_roller_10, origin xyz=0 -0.065 0.000 rpy=0 0 0, axis 0 0 -1
- added joint OmniFL_roller_11_joint: type continuous, parent OmniFL_wheel, child OmniFL_roller_11, origin xyz=0 -0.0761 -0.0247 rpy=0 0 0, axis 0 0.309 -0.951
- added joint OmniFL_roller_12_joint: type continuous, parent OmniFL_wheel, child OmniFL_roller_12, origin xyz=0 -0.0526 -0.0382 rpy=0 0 0, axis 0 0.588 -0.809
- added joint OmniFL_roller_13_joint: type continuous, parent OmniFL_wheel, child OmniFL_roller_13, origin xyz=0 -0.0470 -0.0647 rpy=0 0 0, axis 0 0.809 -0.588
- added joint OmniFL_roller_14_joint: type continuous, parent OmniFL_wheel, child OmniFL_roller_14, origin xyz=0 -0.0201 -0.0617 rpy=0 0 0, axis 0 0.951 -0.309
- added joint OmniFL_roller_15_joint: type continuous, parent OmniFL_wheel, child OmniFL_roller_15, origin xyz=0 0.000 -0.080 rpy=0 0 0, axis 0 1 0
- added joint OmniFL_roller_16_joint: type continuous, parent OmniFL_wheel, child OmniFL_roller_16, origin xyz=0 0.0201 -0.0617 rpy=0 0 0, axis 0 0.951 0.309
- added joint OmniFL_roller_17_joint: type continuous, parent OmniFL_wheel, child OmniFL_roller_17, origin xyz=0 0.0470 -0.0647 rpy=0 0 0, axis 0 0.809 0.588
- added joint OmniFL_roller_18_joint: type continuous, parent OmniFL_wheel, child OmniFL_roller_18, origin xyz=0 0.0526 -0.0382 rpy=0 0 0, axis 0 0.588 0.809
- added joint OmniFL_roller_19_joint: type continuous, parent OmniFL_wheel, child OmniFL_roller_19, origin xyz=0 0.0761 -0.0247 rpy=0 0 0, axis 0 0.309 0.951
- added joint OmniFR_roller_10_joint: type continuous, parent OmniFR_wheel, child OmniFR_roller_10, origin xyz=0 -0.065 0.000 rpy=0 0 0, axis 0 0 -1
- added joint OmniFR_roller_11_joint: type continuous, parent OmniFR_wheel, child OmniFR_roller_11, origin xyz=0 -0.0761 -0.0247 rpy=0 0 0, axis 0 0.309 -0.951
- added joint OmniFR_roller_12_joint: type continuous, parent OmniFR_wheel, child OmniFR_roller_12, origin xyz=0 -0.0526 -0.0382 rpy=0 0 0, axis 0 0.588 -0.809
- added joint OmniFR_roller_13_joint: type continuous, parent OmniFR_wheel, child OmniFR_roller_13, origin xyz=0 -0.0470 -0.0647 rpy=0 0 0, axis 0 0.809 -0.588
- added joint OmniFR_roller_14_joint: type continuous, parent OmniFR_wheel, child OmniFR_roller_14, origin xyz=0 -0.0201 -0.0617 rpy=0 0 0, axis 0 0.951 -0.309
- added joint OmniFR_roller_15_joint: type continuous, parent OmniFR_wheel, child OmniFR_roller_15, origin xyz=0 0.000 -0.080 rpy=0 0 0, axis 0 1 0
- added joint OmniFR_roller_16_joint: type continuous, parent OmniFR_wheel, child OmniFR_roller_16, origin xyz=0 0.0201 -0.0617 rpy=0 0 0, axis 0 0.951 0.309
- added joint OmniFR_roller_17_joint: type continuous, parent OmniFR_wheel, child OmniFR_roller_17, origin xyz=0 0.0470 -0.0647 rpy=0 0 0, axis 0 0.809 0.588
- added joint OmniFR_roller_18_joint: type continuous, parent OmniFR_wheel, child OmniFR_roller_18, origin xyz=0 0.0526 -0.0382 rpy=0 0 0, axis 0 0.588 0.809
- added joint OmniFR_roller_19_joint: type continuous, parent OmniFR_wheel, child OmniFR_roller_19, origin xyz=0 0.0761 -0.0247 rpy=0 0 0, axis 0 0.309 0.951
- added joint OmniR_roller_10_joint: type continuous, parent OmniR_wheel, child OmniR_roller_10, origin xyz=0 -0.065 0.000 rpy=0 0 0, axis 0 0 -1
- added joint OmniR_roller_11_joint: type continuous, parent OmniR_wheel, child OmniR_roller_11, origin xyz=0 -0.0761 -0.0247 rpy=0 0 0, axis 0 0.309 -0.951
- added joint OmniR_roller_12_joint: type continuous, parent OmniR_wheel, child OmniR_roller_12, origin xyz=0 -0.0526 -0.0382 rpy=0 0 0, axis 0 0.588 -0.809
- added joint OmniR_roller_13_joint: type continuous, parent OmniR_wheel, child OmniR_roller_13, origin xyz=0 -0.0470 -0.0647 rpy=0 0 0, axis 0 0.809 -0.588
- added joint OmniR_roller_14_joint: type continuous, parent OmniR_wheel, child OmniR_roller_14, origin xyz=0 -0.0201 -0.0617 rpy=0 0 0, axis 0 0.951 -0.309
- added joint OmniR_roller_15_joint: type continuous, parent OmniR_wheel, child OmniR_roller_15, origin xyz=0 0.000 -0.080 rpy=0 0 0, axis 0 1 0
- added joint OmniR_roller_16_joint: type continuous, parent OmniR_wheel, child OmniR_roller_16, origin xyz=0 0.0201 -0.0617 rpy=0 0 0, axis 0 0.951 0.309
- added joint OmniR_roller_17_joint: type continuous, parent OmniR_wheel, child OmniR_roller_17, origin xyz=0 0.0470 -0.0647 rpy=0 0 0, axis 0 0.809 0.588
- added joint OmniR_roller_18_joint: type continuous, parent OmniR_wheel, child OmniR_roller_18, origin xyz=0 0.0526 -0.0382 rpy=0 0 0, axis 0 0.588 0.809
- added joint OmniR_roller_19_joint: type continuous, parent OmniR_wheel, child OmniR_roller_19, origin xyz=0 0.0761 -0.0247 rpy=0 0 0, axis 0 0.309 0.951
- joint OmniFL_roller_0_joint: origin xyz=0 0.065 0.0 rpy=0 0 0 -> xyz=0 0.065 0.000 rpy=0 0 0
- joint OmniFL_roller_1_joint: axis 0 -0.588 0.809 -> 0 -0.309 0.951; origin xyz=0 0.0526 0.0380 rpy=0 0 0 -> xyz=0 0.0761 0.0247 rpy=0 0 0
- joint OmniFL_roller_2_joint: axis 0 -0.940 0.342 -> 0 -0.588 0.809; origin xyz=0 0.0201 0.0617 rpy=0 0 0 -> xyz=0 0.0526 0.0382 rpy=0 0 0
- joint OmniFL_roller_3_joint: axis 0 -0.940 -0.342 -> 0 -0.809 0.588; origin xyz=0 -0.0201 0.0617 rpy=0 0 0 -> xyz=0 0.0470 0.0647 rpy=0 0 0
- joint OmniFL_roller_4_joint: axis 0 -0.588 -0.809 -> 0 -0.951 0.309; origin xyz=0 -0.0526 0.0380 rpy=0 0 0 -> xyz=0 0.0201 0.0617 rpy=0 0 0
- joint OmniFL_roller_5_joint: axis 0 0 -1 -> 0 -1 0; origin xyz=0 -0.065 0.0 rpy=0 0 0 -> xyz=0 0.000 0.080 rpy=0 0 0
- joint OmniFL_roller_6_joint: axis 0 0.588 -0.809 -> 0 -0.951 -0.309; origin xyz=0 -0.0526 -0.0380 rpy=0 0 0 -> xyz=0 -0.0201 0.0617 rpy=0 0 0
- joint OmniFL_roller_7_joint: axis 0 0.940 -0.342 -> 0 -0.809 -0.588; origin xyz=0 -0.0201 -0.0617 rpy=0 0 0 -> xyz=0 -0.0470 0.0647 rpy=0 0 0
- joint OmniFL_roller_8_joint: axis 0 0.940 0.342 -> 0 -0.588 -0.809; origin xyz=0 0.0201 -0.0617 rpy=0 0 0 -> xyz=0 -0.0526 0.0382 rpy=0 0 0
- joint OmniFL_roller_9_joint: axis 0 0.588 0.809 -> 0 -0.309 -0.951; origin xyz=0 0.0526 -0.0380 rpy=0 0 0 -> xyz=0 -0.0761 0.0247 rpy=0 0 0
- joint OmniFR_roller_0_joint: origin xyz=0 0.065 0.0 rpy=0 0 0 -> xyz=0 0.065 0.000 rpy=0 0 0
- joint OmniFR_roller_1_joint: axis 0 -0.588 0.809 -> 0 -0.309 0.951; origin xyz=0 0.0526 0.0380 rpy=0 0 0 -> xyz=0 0.0761 0.0247 rpy=0 0 0
- joint OmniFR_roller_2_joint: axis 0 -0.940 0.342 -> 0 -0.588 0.809; origin xyz=0 0.0201 0.0617 rpy=0 0 0 -> xyz=0 0.0526 0.0382 rpy=0 0 0
- joint OmniFR_roller_3_joint: axis 0 -0.940 -0.342 -> 0 -0.809 0.588; origin xyz=0 -0.0201 0.0617 rpy=0 0 0 -> xyz=0 0.0470 0.0647 rpy=0 0 0
- joint OmniFR_roller_4_joint: axis 0 -0.588 -0.809 -> 0 -0.951 0.309; origin xyz=0 -0.0526 0.0380 rpy=0 0 0 -> xyz=0 0.0201 0.0617 rpy=0 0 0
- joint OmniFR_roller_5_joint: axis 0 0 -1 -> 0 -1 0; origin xyz=0 -0.065 0.0 rpy=0 0 0 -> xyz=0 0.000 0.080 rpy=0 0 0
- joint OmniFR_roller_6_joint: axis 0 0.588 -0.809 -> 0 -0.951 -0.309; origin xyz=0 -0.0526 -0.0380 rpy=0 0 0 -> xyz=0 -0.0201 0.0617 rpy=0 0 0
- joint OmniFR_roller_7_joint: axis 0 0.940 -0.342 -> 0 -0.809 -0.588; origin xyz=0 -0.0201 -0.0617 rpy=0 0 0 -> xyz=0 -0.0470 0.0647 rpy=0 0 0
- joint OmniFR_roller_8_joint: axis 0 0.940 0.342 -> 0 -0.588 -0.809; origin xyz=0 0.0201 -0.0617 rpy=0 0 0 -> xyz=0 -0.0526 0.0382 rpy=0 0 0
- joint OmniFR_roller_9_joint: axis 0 0.588 0.809 -> 0 -0.309 -0.951; origin xyz=0 0.0526 -0.0380 rpy=0 0 0 -> xyz=0 -0.0761 0.0247 rpy=0 0 0
- joint OmniR_roller_0_joint: origin xyz=0 0.065 0.0 rpy=0 0 0 -> xyz=0 0.065 0.000 rpy=0 0 0
- joint OmniR_roller_1_joint: axis 0 -0.588 0.809 -> 0 -0.309 0.951; origin xyz=0 0.0526 0.0380 rpy=0 0 0 -> xyz=0 0.0761 0.0247 rpy=0 0 0
- joint OmniR_roller_2_joint: axis 0 -0.940 0.342 -> 0 -0.588 0.809; origin xyz=0 0.0201 0.0617 rpy=0 0 0 -> xyz=0 0.0526 0.0382 rpy=0 0 0
- joint OmniR_roller_3_joint: axis 0 -0.940 -0.342 -> 0 -0.809 0.588; origin xyz=0 -0.0201 0.0617 rpy=0 0 0 -> xyz=0 0.0470 0.0647 rpy=0 0 0
- joint OmniR_roller_4_joint: axis 0 -0.588 -0.809 -> 0 -0.951 0.309; origin xyz=0 -0.0526 0.0380 rpy=0 0 0 -> xyz=0 0.0201 0.0617 rpy=0 0 0
- joint OmniR_roller_5_joint: axis 0 0 -1 -> 0 -1 0; origin xyz=0 -0.065 0.0 rpy=0 0 0 -> xyz=0 0.000 0.080 rpy=0 0 0
- joint OmniR_roller_6_joint: axis 0 0.588 -0.809 -> 0 -0.951 -0.309; origin xyz=0 -0.0526 -0.0380 rpy=0 0 0 -> xyz=0 -0.0201 0.0617 rpy=0 0 0
- joint OmniR_roller_7_joint: axis 0 0.940 -0.342 -> 0 -0.809 -0.588; origin xyz=0 -0.0201 -0.0617 rpy=0 0 0 -> xyz=0 -0.0470 0.0647 rpy=0 0 0
- joint OmniR_roller_8_joint: axis 0 0.940 0.342 -> 0 -0.588 -0.809; origin xyz=0 0.0201 -0.0617 rpy=0 0 0 -> xyz=0 -0.0526 0.0382 rpy=0 0 0
- joint OmniR_roller_9_joint: axis 0 0.588 0.809 -> 0 -0.309 -0.951; origin xyz=0 0.0526 -0.0380 rpy=0 0 0 -> xyz=0 -0.0761 0.0247 rpy=0 0 0

Commit message: 1. Joint limit change 2. Rotation is not working 3. Should I divided manipulation and navigation?

File: anubis/anubis_omni.urdf (robot description, URDF)
Before this commit: robot anubis, 84 links, 83 joints
Links:
- link OmniFL_wheel: mass 4 -> 1.5
- link OmniFR_wheel: mass 4 -> 1.5
- link OmniR_wheel: mass 4 -> 1.5
- link base_link: mass 30 -> 20

Commit message: small mass for dummy spheres were the problem 1. Fix rotation

File: anubis/anubis_omni.urdf (robot description, URDF)
Before this commit: robot anubis, 84 links, 83 joints
Links:
- link OmniFL_roller_0: mass 0.05 -> 3
- link OmniFL_roller_1: mass 0.01 -> 2
- link OmniFL_roller_10: mass 0.05 -> 3
- link OmniFL_roller_11: mass 0.01 -> 2
- link OmniFL_roller_12: mass 0.05 -> 3
- link OmniFL_roller_13: mass 0.01 -> 2
- link OmniFL_roller_14: mass 0.05 -> 3
- link OmniFL_roller_15: mass 0.01 -> 2
- link OmniFL_roller_16: mass 0.05 -> 3
- link OmniFL_roller_17: mass 0.01 -> 2
- link OmniFL_roller_18: mass 0.05 -> 3
- link OmniFL_roller_19: mass 0.01 -> 2
- link OmniFL_roller_2: mass 0.05 -> 3
- link OmniFL_roller_3: mass 0.01 -> 2
- link OmniFL_roller_4: mass 0.05 -> 3
- link OmniFL_roller_5: mass 0.01 -> 2
- link OmniFL_roller_6: mass 0.05 -> 3
- link OmniFL_roller_7: mass 0.01 -> 2
- link OmniFL_roller_8: mass 0.05 -> 3
- link OmniFL_roller_9: mass 0.01 -> 2
- link OmniFL_wheel: mass 1.5 -> 3.1
- link OmniFR_roller_0: mass 0.05 -> 3
- link OmniFR_roller_1: mass 0.01 -> 2
- link OmniFR_roller_10: mass 0.05 -> 3
- link OmniFR_roller_11: mass 0.01 -> 2
- link OmniFR_roller_12: mass 0.05 -> 3
- link OmniFR_roller_13: mass 0.01 -> 2
- link OmniFR_roller_14: mass 0.05 -> 3
- link OmniFR_roller_15: mass 0.01 -> 2
- link OmniFR_roller_16: mass 0.05 -> 3
- link OmniFR_roller_17: mass 0.01 -> 2
- link OmniFR_roller_18: mass 0.05 -> 3
- link OmniFR_roller_19: mass 0.01 -> 2
- link OmniFR_roller_2: mass 0.05 -> 3
- link OmniFR_roller_3: mass 0.01 -> 2
- link OmniFR_roller_4: mass 0.05 -> 3
- link OmniFR_roller_5: mass 0.01 -> 2
- link OmniFR_roller_6: mass 0.05 -> 3
- link OmniFR_roller_7: mass 0.01 -> 2
- link OmniFR_roller_8: mass 0.05 -> 3
- link OmniFR_roller_9: mass 0.01 -> 2
- link OmniFR_wheel: mass 1.5 -> 3.1
- link OmniR_roller_0: mass 0.05 -> 3
- link OmniR_roller_1: mass 0.01 -> 2
- link OmniR_roller_10: mass 0.05 -> 3
- link OmniR_roller_11: mass 0.01 -> 2
- link OmniR_roller_12: mass 0.05 -> 3
- link OmniR_roller_13: mass 0.01 -> 2
- link OmniR_roller_14: mass 0.05 -> 3
- link OmniR_roller_15: mass 0.01 -> 2
- link OmniR_roller_16: mass 0.05 -> 3
- link OmniR_roller_17: mass 0.01 -> 2
- link OmniR_roller_18: mass 0.05 -> 3
- link OmniR_roller_19: mass 0.01 -> 2
- link OmniR_roller_2: mass 0.05 -> 3
- link OmniR_roller_3: mass 0.01 -> 2
- link OmniR_roller_4: mass 0.05 -> 3
- link OmniR_roller_5: mass 0.01 -> 2
- link OmniR_roller_6: mass 0.05 -> 3
- link OmniR_roller_7: mass 0.01 -> 2
- link OmniR_roller_8: mass 0.05 -> 3
- link OmniR_roller_9: mass 0.01 -> 2
- link OmniR_wheel: mass 1.5 -> 3.1
- link base_link: mass 20 -> 15
Joints:
- joint arm1_base_link_joint: limit lower=-1.74533 upper=1.74533 effort=39 velocity=1.3963 -> lower=-0.523599 upper= 0.523599 effort=3 velocity=1.3963
- joint arm2_base_link_joint: limit lower=-1.74533 upper=1.74533 effort=39 velocity=1.3963 -> lower=-0.523599 upper=0.523599 effort=3 velocity=1.3963
- joint link11_joint: limit lower=-0.523599 upper=0.523599 effort=39 velocity=1.3963 -> lower=-0.74533 upper=1.91986 effort=3 velocity=1.3963
- joint link12_joint: limit lower=-0.523599 upper=1.91986 effort=39 velocity=1.3963 -> lower=0.174533 upper=2.79253 effort=3 velocity=1.3963
- joint link13_joint: limit lower=0.174533 upper=2.79253 effort=39 velocity=1.3963 -> lower=-1.5708 upper=1.74533 effort=3 velocity=1.3963
- joint link14_joint: limit lower=-1.5708 upper=1.74533 effort=39 velocity=1.3963 -> lower=-1.5708 upper=1.57085 effort=3 velocity=1.3963
- joint link15_joint: limit lower=-1.5708 upper=1.57085 effort=39 velocity=1.3963 -> lower=-1.74533 upper=1.74533 effort=3 velocity=1.3963
- joint link21_joint: limit lower=-0.523599 upper=0.523599 effort=39 velocity=1.3963 -> lower=-0.74533 upper=1.91986 effort=3 velocity=1.3963
- joint link22_joint: limit lower=-0.523599 upper=1.91986 effort=39 velocity=1.3963 -> lower=-0.174533 upper=2.79253 effort=3 velocity=1.3963
- joint link23_joint: limit lower=0.174533 upper=2.79253 effort=39 velocity=1.3963 -> lower=-1.5708 upper=1.74533 effort=3 velocity=1.3963
- joint link24_joint: limit lower=-1.5708 upper=1.74533 effort=39 velocity=1.3963 -> lower=-1.5708 upper=1.5708 effort=3 velocity=1.3963
- joint link25_joint: limit lower=-1.5708 upper=1.57085 effort=39 velocity=1.3963 -> lower=-1.74533 upper=1.74533 effort=3 velocity=1.3963

Commit message: Need to check if vr_headset_frame is well defined in isaacsim streaming

File: anubis/anubis_omni.urdf (robot description, URDF)
Before this commit: robot anubis, 84 links, 83 joints
Links:
- added link vr_headset_frame
- link arm1_base_link: mass None -> 1
- link arm2_base_link: mass None -> 1
- link link11: mass 0.0608351104988555 -> 0.608351104988555
Joints:
- added joint vr_headset_joint: type fixed, parent base_link, child vr_headset_frame, origin xyz=0 0 1.5 rpy=-0.52 0 0

Commit message: [absolute control] damping and stiffness need to be checked

File: anubis/anubis_omni.urdf (robot description, URDF)
Before this commit: robot anubis, 85 links, 84 joints
Joints:
- joint vr_headset_joint: origin xyz=0 0 1.5 rpy=-0.52 0 0 -> xyz=-0.15 0 1.4 rpy=0 0 -1.5708

Commit message: Maybe change to operational space controller

File: anubis/anubis_omni.urdf (robot description, URDF)
Before this commit: robot anubis, 85 links, 84 joints
Links:
- link arm1_base_link: mass 1 -> 0.05
- link arm2_base_link: mass 1 -> 0.05
- link ee_link1: mass 0.0062357399313257 -> 0.05
- link ee_link2: mass 0.0062357399313257 -> 0.05
- link gripper1L: mass 0.925 -> 0.05
- link gripper1R: mass 0.925 -> 0.05
- link gripper2L: mass 0.925 -> 0.05
- link gripper2R: mass 0.925 -> 0.05
- link gripper2_base_link: mass 0.62357399313257 -> 0.05
- link gripper_base_link: mass 0.62357399313257 -> 0.05
- link link11: mass 0.608351104988555 -> 0.05
- link link12: mass 1.0733279014126 -> 0.5
- link link13: mass 0.499404738025019 -> 0.05
- link link14: mass 0.0809712553169999 -> 0.05
- link link15: mass 0.602357399313257 -> 0.05
- link link21: mass 0.0608351104988555 -> 0.05
- link link22: mass 1.0733279014126 -> 0.5
- link link23: mass 0.499404738025019 -> 0.05
- link link24: mass 0.0809712553169999 -> 0.05
- link link25: mass 0.602357399313257 -> 0.05

Commit message: 1. right finger is stronger Right finger is really just going to the closed command expr 2. More friction on mobile base?

File: anubis/anubis_omni.urdf (robot description, URDF)
Before this commit: robot anubis, 85 links, 84 joints
Links:
- link gripper1L: geometry collision box size=0.018 0.035 0.093; visual mesh filename=package://anubis/meshes/gripper/fingerL.stl
- link gripper1R: geometry collision box size=0.018 0.035 0.093; visual mesh filename=package://anubis/meshes/gripper/fingerR.stl
- link gripper2L: geometry collision box size=0.018 0.035 0.093; visual mesh filename=package://anubis/meshes/gripper/fingerL.stl
- link gripper2R: geometry collision box size=0.018 0.035 0.093; visual mesh filename=package://anubis/meshes/gripper/fingerR.stl
Joints:
- joint gripper1R_joint: mimic joint=gripper1_joint multiplier=1 offset=0 -> (none)
- joint gripper2R_joint: mimic joint=gripper2_joint multiplier=1 offset=0 -> (none)

Commit message: When the cabinet is heavy or light, shouldn't the action be different?

File: anubis/anubis_omni.urdf (robot description, URDF)
Before this commit: robot anubis, 85 links, 84 joints
Joints:
- joint gripper1R_joint: limit lower=0 upper=0.04 effort=1 velocity=4.8 -> lower=0 upper=0.04 effort=4 velocity=4.8; mimic (none) -> joint=gripper1_joint multiplier=1 offset=0
- joint gripper1_joint: limit lower=0 upper=0.04 effort=1 velocity=4.8 -> lower=0 upper=0.04 effort=4 velocity=4.8
- joint gripper2R_joint: limit lower=0 upper=0.04 effort=1 velocity=4.8 -> lower=0 upper=0.04 effort=4 velocity=4.8; mimic (none) -> joint=gripper2_joint multiplier=1 offset=0
- joint gripper2_joint: limit lower=0 upper=0.04 effort=1 velocity=4.8 -> lower=0 upper=0.04 effort=4 velocity=4.8
