Commit message: why the top drawer is not moving how to handle big external force

File: anubis/anubis_omni.urdf (robot description, URDF)
Before this commit: robot anubis, 85 links, 84 joints
Links:
- link OmniFL_roller_0: mass 3 -> 0.5
- link OmniFL_roller_1: mass 2 -> 0.5
- link OmniFL_roller_10: mass 3 -> 0.5
- link OmniFL_roller_11: mass 2 -> 0.5
- link OmniFL_roller_12: mass 3 -> 0.5
- link OmniFL_roller_13: mass 2 -> 0.5
- link OmniFL_roller_14: mass 3 -> 0.5
- link OmniFL_roller_15: mass 2 -> 0.5
- link OmniFL_roller_16: mass 3 -> 0.5
- link OmniFL_roller_17: mass 2 -> 0.5
- link OmniFL_roller_18: mass 3 -> 0.5
- link OmniFL_roller_19: mass 2 -> 0.5
- link OmniFL_roller_2: mass 3 -> 0.5
- link OmniFL_roller_3: mass 2 -> 0.5
- link OmniFL_roller_4: mass 3 -> 0.5
- link OmniFL_roller_5: mass 2 -> 0.5
- link OmniFL_roller_6: mass 3 -> 0.5
- link OmniFL_roller_7: mass 2 -> 0.5
- link OmniFL_roller_8: mass 3 -> 0.5
- link OmniFL_roller_9: mass 2 -> 0.5
- link OmniFL_wheel: mass 3.1 -> 0.5
- link OmniFR_roller_0: mass 3 -> 0.5
- link OmniFR_roller_1: mass 2 -> 0.5
- link OmniFR_roller_10: mass 3 -> 0.5
- link OmniFR_roller_11: mass 2 -> 0.5
- link OmniFR_roller_12: mass 3 -> 0.5
- link OmniFR_roller_13: mass 2 -> 0.5
- link OmniFR_roller_14: mass 3 -> 0.5
- link OmniFR_roller_15: mass 2 -> 0.5
- link OmniFR_roller_16: mass 3 -> 0.5
- link OmniFR_roller_17: mass 2 -> 0.5
- link OmniFR_roller_18: mass 3 -> 0.5
- link OmniFR_roller_19: mass 2 -> 0.5
- link OmniFR_roller_2: mass 3 -> 0.5
- link OmniFR_roller_3: mass 2 -> 0.5
- link OmniFR_roller_4: mass 3 -> 0.5
- link OmniFR_roller_5: mass 2 -> 0.5
- link OmniFR_roller_6: mass 3 -> 0.5
- link OmniFR_roller_7: mass 2 -> 0.5
- link OmniFR_roller_8: mass 3 -> 0.5
- link OmniFR_roller_9: mass 2 -> 0.5
- link OmniFR_wheel: mass 3.1 -> 0.5
- link OmniR_roller_0: mass 3 -> 0.5
- link OmniR_roller_1: mass 2 -> 0.5
- link OmniR_roller_10: mass 3 -> 0.5
- link OmniR_roller_11: mass 2 -> 0.5
- link OmniR_roller_12: mass 3 -> 0.5
- link OmniR_roller_13: mass 2 -> 0.5
- link OmniR_roller_14: mass 3 -> 0.5
- link OmniR_roller_15: mass 2 -> 0.5
- link OmniR_roller_16: mass 3 -> 0.5
- link OmniR_roller_17: mass 2 -> 0.5
- link OmniR_roller_18: mass 3 -> 0.5
- link OmniR_roller_19: mass 2 -> 0.5
- link OmniR_roller_2: mass 3 -> 0.5
- link OmniR_roller_3: mass 2 -> 0.5
- link OmniR_roller_4: mass 3 -> 0.5
- link OmniR_roller_5: mass 2 -> 0.5
- link OmniR_roller_6: mass 3 -> 0.5
- link OmniR_roller_7: mass 2 -> 0.5
- link OmniR_roller_8: mass 3 -> 0.5
- link OmniR_roller_9: mass 2 -> 0.5
- link OmniR_wheel: mass 3.1 -> 2.5
- link arm1_base_link: mass 0.05 -> 0.641
- link arm2_base_link: mass 0.05 -> 0.641
- link base_link: mass 15 -> 50
- link ee_link1: mass 0.05 ->  0.300
- link ee_link2: mass 0.05 ->  0.300
- link gripper1L: mass 0.05 -> 0.7
- link gripper1R: mass 0.05 -> 0.7
- link gripper2L: mass 0.05 -> 0.7
- link gripper2R: mass 0.05 -> 0.7
- link gripper2_base_link: mass 0.05 -> 0.400
- link gripper_base_link: mass 0.05 -> 0.400
- link link11: mass 0.05 -> 1.700
- link link12: mass 0.5 -> 1.150
- link link13: mass 0.05 ->  1.200
- link link14: mass 0.05 -> 0.800
- link link15: mass 0.05 -> 0.800
- link link21: mass 0.05 ->  1.700
- link link22: mass 0.5 -> 1.150
- link link23: mass 0.05 ->  1.200
- link link24: mass 0.05 -> 0.800
- link link25: mass 0.05 -> 0.800
